File: Project-ESD-Final-V/Project-ESD/Project-ESD.kicad_pcb (KiCad board)
At the start: 2 copper layers, 70 x 90 mm, 57 parts, among them J1 USB_OTG, J2 Conn_01x05_Male, J3 Conn_01x02_Female, J4 Conn_Coaxial, J5 Conn_01x07_Male, J6 Conn_01x02_Female, SW1 SW_Push, SW10 SW_Push, SW11 SW_Push, SW12 SW_Push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

Commit message: Final verson 2
Parts:
- R2: value 6.8k -> 5.6k
- moved J4 3.30 mm to (127.0, 69.6), turned to 90 degrees
- moved C8 1.27 mm to (141.3, 70.6)
- moved C14 1.27 mm to (138.3, 69.6)
- moved C15 1.27 mm to (135.3, 70.6)
Routing:
- net +3V3: track 195.9 -> 204.2 mm
- net +5V: track 30.5 -> 35.0 mm
- net GND: track 89.1 -> 86.0 mm, vias 78 -> 92
- net Net-(C14-Pad2): track 9.80 -> 9.27 mm
