File: Project-ESD-Final-V/Project-ESD/Project-ESD.sch (KiCad schematic (older format))
At the start: 57 parts, among them J1 USB_OTG, J2 Conn_01x05_Male, J3 Conn_01x02_Female, J4 Conn_Coaxial, J5 Conn_01x07_Male, J6 Conn_01x02_Female, SW1 SW_Push, SW10 SW_Push, SW11 SW_Push, SW12 SW_Push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

Commit message: Final verson 2
Parts:
- R2: value 6.8k -> 5.6k
Changed lines of the file:
@@
 P 4350 1400
 F 0 "R2" H 4420 1446 50  0000 L CNN
-F 1 "6.8k" H 4420 1355 50  0000 L CNN
+F 1 "5.6k" H 4420 1355 50  0000 L CNN
 F 2 "Resistor_SMD:R_0805_2012Metric_Pad1.15x1.40mm_HandSolder" V 4280 1400 50  0001 C CNN
 F 3 "~" H 4350 1400 50  0001 C CNN
